Commit message: adding colliders to urdf

File: resources/mushr_description/robots/racecar-mit-phys.urdf (robot description, URDF)
Before this commit: robot racecar, 9 links, 8 joints
Links:
- link back_left_wheel: geometry collision cylinder length=0.045 radius=0.05; visual cylinder length=0.045 radius=0.05
- link back_right_wheel: geometry collision cylinder length=0.045 radius=0.05; visual cylinder length=0.045 radius=0.05
- link chassis: geometry collision box size=0.325 0.2 0.1; visual box size=0.325 0.2 0.1
- link front_left_wheel: geometry collision cylinder length=0.045 radius=0.05; visual cylinder length=0.045 radius=0.05
- link front_right_wheel: mass None -> 1; geometry collision cylinder length=0.045 radius=0.05; visual cylinder length=0.045 radius=0.05

File: resources/mushr_description/robots/racecar-mit-phys.urdf.xacro (robot description, xacro)
@@ -3,9 +3,5 @@
 <!-- A simple model of the racecar for rviz -->
 <robot xmlns:xacro="http://www.ros.org/wiki/xacro" name="racecar">
-  <xacro:macro name="inertial_block" params="mass">
-    <inertial>
-      <mass value="${mass}"/>
-    </inertial>
-  </xacro:macro>
+  <!-- GEOMETRY PARAMS -->
   <xacro:property name="wheelbase" value="0.325" />
   <xacro:property name="width" value="0.2" />
@@ -49,4 +45,37 @@
     <color rgba="0.3 0.57 1. 1."/>
   </material>
+  <!-- MACROS -->
+  <xacro:macro name="wheel_block" params="name">
+    <link name="${name}">
+      <xacro:visual_collision_block>
+        <cylinder radius="${wheel_radius}" length="${wheel_length}"/>
+        <container>
+          <material name="black"/>
+          <origin rpy="${pi/2} 0 0"/>
+        </container>
+      </xacro:visual_collision_block>
+      <xacro:inertial_block mass="${wheel_mass}"/>
+    </link>
+  </xacro:macro>
+  <xacro:macro name="inertial_block" params="mass">
+    <inertial>
+      <mass value="${mass}"/>
+    </inertial>
+  </xacro:macro>
+  <xacro:macro name="visual_collision_block" params="*geometry **kwargs">
+    <visual>
+      <geometry>
+        <xacro:insert_block name="geometry"/>
+      </geometry>
+      <xacro:insert_block name="kwargs"/>
+    </visual>
+    <collision>
+      <geometry>
+        <xacro:insert_block name="geometry"/>
+      </geometry>
+      <xacro:insert_block name="kwargs"/>
+    </collision>
+  </xacro:macro>
+  <!-- MAIN FILE -->
 	<link name="base">
     <visual>
@@ -73,4 +102,9 @@
       <material name="blue"/>
     </visual>
+    <collision>
+      <geometry>
+        <box size="${wheelbase} ${width} ${height}"/>
+      </geometry>
+    </collision>
     <xacro:inertial_block mass="${chassis_mass}"/>
   </link>
@@ -100,14 +134,5 @@
     <xacro:insert_block name="wheel_joint_props"/>
   </joint>
-  <link name="back_left_wheel">
-    <visual>
-      <geometry>
-        <cylinder radius="${wheel_radius}" length="${wheel_length}"/>
-      </geometry>
-      <material name="black"/>
-      <origin rpy="${pi/2} 0 0"/>
-    </visual>
-    <xacro:inertial_block mass="${wheel_mass}"/>
-  </link>
+  <xacro:wheel_block name="back_left_wheel"/>
   <joint name="chassis_to_back_right_wheel" type="continuous">
     <parent link="chassis"/>
@@ -116,14 +141,5 @@
     <xacro:insert_block name="wheel_joint_props"/>
   </joint>
-  <link name="back_right_wheel">
-    <visual>
-      <geometry>
-        <cylinder radius="${wheel_radius}" length="${wheel_length}"/>
-      </geometry>
-      <material name="black"/>
-      <origin rpy="${pi/2} 0 0"/>
-    </visual>
-    <xacro:inertial_block mass="${wheel_mass}"/>
-  </link>
+  <xacro:wheel_block name="back_right_wheel"/>
   <joint name="chassis_to_front_left_hinge" type="revolute">
     <parent link="chassis"/>
@@ -140,14 +156,5 @@
     <xacro:insert_block name="wheel_joint_props"/>
   </joint>
-  <link name="front_left_wheel">
-    <visual>
-      <geometry>
-        <cylinder radius="${wheel_radius}" length="${wheel_length}"/>
-      </geometry>
-      <material name="black"/>
-      <origin rpy="${pi/2} 0 0"/>
-    </visual>
-    <xacro:inertial_block mass="${wheel_mass}"/>
-  </link>
+  <xacro:wheel_block name="front_left_wheel"/>
   <joint name="chassis_to_front_right_hinge" type="revolute">
     <parent link="chassis"/>
@@ -164,13 +171,4 @@
     <xacro:insert_block name="wheel_joint_props"/>
   </joint>
-  <link name="front_right_wheel">
-    <visual>
-      <geometry>
-        <cylinder radius="${wheel_radius}" length="${wheel_length}"/>
-      </geometry>
-      <material name="black"/>
-      <origin rpy="${pi/2} 0 0"/>
-    </visual>
-    <!-- <xacro:inertial_block mass="${wheel_mass}"/> -->
-  </link>
+  <xacro:wheel_block name="front_right_wheel"/>
 </robot>

Commit message: vehicles moving forward in environment

File: resources/mushr_description/robots/racecar-mit-phys.urdf (robot description, URDF)
Before this commit: robot racecar, 9 links, 8 joints
Links:
- removed link base
- link back_left_wheel: mass 1 -> 0.5
- link back_right_wheel: mass 1 -> 0.5
- link chassis: mass 1 -> 10; geometry visual box size=0.325 0.2 0.1
- link front_left_wheel: mass 1 -> 0.5
- link front_right_wheel: mass 1 -> 0.5
- link laser_model: mass 1 -> 0.01
Joints:
- removed joint base_to_chassis
- joint chassis_to_back_left_wheel: type continuous -> revolute
- joint chassis_to_back_right_wheel: type continuous -> revolute
- joint chassis_to_front_left_hinge: limit (none) -> lower=-0.5235987755982988 upper=0.5235987755982988 effort=1000 velocity=1.0
- joint chassis_to_front_right_hinge: limit (none) -> lower=-0.5235987755982988 upper=0.5235987755982988 effort=1000 velocity=1.0

File: resources/mushr_description/robots/racecar-mit-phys.urdf.xacro (robot description, xacro)
@@ -15,7 +15,10 @@
   <!-- ISAAC GYM RIGID BODY PARAMS -->
   <!-- Wheel Properties -->
-  <xacro:property name="wheel_mass" value="1" />
+  <xacro:property name="wheel_mass" value=".5" />
   <xacro:property name="wheel_joint_props">
     <axis xyz="0 1 0"/>
+  </xacro:property>
+  <xacro:property name="wheel_inertia">
+    <inertia ixx="0.0013" ixy="0" ixz="0" iyy="0.0024" iyz="0" izz="0.0013"/>
   </xacro:property>
   <!-- Hinge Properties -->
@@ -23,8 +26,8 @@
   <xacro:property name="hinge_joint_props">
     <axis xyz="0 0 1"/>
-    <!-- <limit lower="${-1 * pi / 6}" upper="${pi / 6}" effort=1000/> -->
+    <limit lower="${-1 * pi / 6}" upper="${pi / 6}" effort="1000" velocity="1.0"/>
   </xacro:property>
   <!-- Chassis Properties -->
-  <xacro:property name="chassis_mass" value="1" />
+  <xacro:property name="chassis_mass" value="10" />
   <xacro:property name="chassis_inertia">
     <inertia
@@ -38,5 +41,5 @@
   </xacro:property>
   <!-- Sensor Properties -->
-  <xacro:property name="laser_mass" value="1" />
+  <xacro:property name="laser_mass" value=".01" />
   <material name="black">
     <color rgba="0.2 0.2 0.2 1."/>
@@ -55,10 +58,15 @@
         </container>
       </xacro:visual_collision_block>
-      <xacro:inertial_block mass="${wheel_mass}"/>
+      <xacro:inertial_block mass="${wheel_mass}">
+        <container>
+          <xacro:insert_block name="wheel_inertia"/>
+        </container>
+      </xacro:inertial_block>
     </link>
   </xacro:macro>
-  <xacro:macro name="inertial_block" params="mass">
+  <xacro:macro name="inertial_block" params="mass **kwargs">
     <inertial>
       <mass value="${mass}"/>
+      <xacro:insert_block name="kwargs"/>
     </inertial>
   </xacro:macro>
@@ -78,20 +86,4 @@
   </xacro:macro>
   <!-- MAIN FILE -->
-	<link name="base">
-    <visual>
-      <origin rpy="0 0 0" xyz="0 0 0"/>
-      <geometry>
-        <box size="0.001 0.001 0.001"/>
-      </geometry>
-    </visual>
-		<!-- <inertial>
-			<origin
-				xyz="0 0 0"
-				rpy="0 0 0" />
-			<mass
-				value="0.1" />
-      <xacro:insert_block name="chassis_inertia"/>
-		</inertial> -->
-	</link>
   <link name="chassis">
     <visual>
@@ -102,16 +94,16 @@
       <material name="blue"/>
     </visual>
-    <collision>
+    <!-- <collision>
       <geometry>
         <box size="${wheelbase} ${width} ${height}"/>
       </geometry>
-    </collision>
-    <xacro:inertial_block mass="${chassis_mass}"/>
+    </collision> -->
+    <xacro:inertial_block mass="${chassis_mass}">
+      <container>
+        <xacro:insert_block name="chassis_inertia"/>
+        <origin xyz="${wheelbase/2} 0 ${ground_offset+height/2}"/>
+      </container>
+    </xacro:inertial_block>
   </link>
-  <joint name="base_to_chassis" type="fixed">
-    <origin rpy="0 0 0" xyz="0 0 0"/>
-    <parent link="base"/>
-    <child link="chassis"/>
-  </joint>
   <joint name="chassis_to_laser_model" type="fixed">
     <parent link="chassis"/>
@@ -126,5 +118,5 @@
       <material name="black"/>
     </visual>
-    <xacro:inertial_block mass="${laser_mass}"/>
+    <xacro:inertial_block mass="${laser_mass}"><container/></xacro:inertial_block>
   </link>
   <joint name="chassis_to_back_left_wheel" type="continuous">
@@ -149,7 +141,7 @@
   </joint>
   <link name="front_left_hinge">
-    <xacro:inertial_block mass="${hinge_mass}"/>
+    <xacro:inertial_block mass="${hinge_mass}"><container/></xacro:inertial_block>
   </link>
-  <joint name="front_left_hinge_to_wheel" type="revolute">
+  <joint name="front_left_hinge_to_wheel" type="continuous">
     <parent link="front_left_hinge"/>
     <child link="front_left_wheel"/>
@@ -164,7 +156,7 @@
   </joint>
   <link name="front_right_hinge">
-    <xacro:inertial_block mass="${hinge_mass}"/>
+     <xacro:inertial_block mass="${hinge_mass}"><container/></xacro:inertial_block>
   </link>
-  <joint name="front_right_hinge_to_wheel" type="revolute">
+  <joint name="front_right_hinge_to_wheel" type="continuous">
     <parent link="front_right_hinge"/>
     <child link="front_right_wheel"/>
